Commit message: fixing tf2 tree for multiple robots

File: chair_ws/src/chair/urdf/airchair.urdf.xacro (robot description, xacro)
@@ -6,5 +6,5 @@
         It now has a target
         It now tilts the camera
-	Version 1.2.
+	Version 1.2a.
 	-->
 <robot name="$(arg name)" xmlns:xacro="http://www.ros.org/wiki/xacro">
@@ -158,10 +158,10 @@
   </gazebo>
   <!-- Left wheel -->
-  <link name="left_wheel_link">
+  <link name="left_wheel">
     <visual>
       <!-- origin rpy="0 1.5708 0" xyz="0 0 0" -->
       <geometry>
         <cylinder length="${robot_wheel_width}" radius="${robot_wheel_radius}" />
-        <!-- mesh filename="$(find chair)/rearwheel.obj" scale="0.001 0.001 0.001"-->>
+        <!-- mesh filename="$(find chair)/rearwheel.obj" scale="0.001 0.001 0.001"-->
       </geometry>
     </visual>
@@ -176,5 +176,5 @@
     <axis xyz="0 0 1" />
     <parent link="base_link" />
-    <child link="left_wheel_link" />
+    <child link="left_wheel" />
     <origin rpy="-1.5708 0 0" xyz="${robot_wheel_xoffset} ${robot_base_width/2+robot_wheel_width/2} ${robot_wheel_zoffset}" />
   </joint>
@@ -326,6 +326,6 @@
       <publish_odom_tf>true</publish_odom_tf>
       <publish_wheel_tf>true</publish_wheel_tf>
-      <odometry_frame>odom</odometry_frame>
-      <robot_base_frame>base_footprint</robot_base_frame>
+      <odometry_frame>${robot_name}/odom</odometry_frame>
+      <robot_base_frame>${robot_name}/base_footprint</robot_base_frame>
       <command_topic>cmd_vel</command_topic>
     </plugin>
